Commit message: changes in file_struct

File: arm_description/urdf/arm.xacro (robot description, xacro)
@@ -1,4 +1,4 @@
 <?xml version="1.0" ?>
-<robot name="mrm" xmlns:xacro="http://www.ros.org/wiki/xacro">
+<robot name="arm" xmlns:xacro="http://www.ros.org/wiki/xacro">
 <!-- BGN - Include -->
 <xacro:include filename="$(find arm_description)/urdf/robot_parameters.xacro" />
@@ -67,7 +67,64 @@
     length="0.25" />
 <!-- END - Robot description -->
+<!-- joint controller gazebo -->
+<transmission name="${link_00_name}_trans">
+    <type>transmission_interface/SimpleTransmission</type>
+    <joint name="${link_00_name}__${link_01_name}">
+        <hardwareInterface>hardware_interface/PositionJointInterface</hardwareInterface>
+    </joint>
+    <actuator name="${link_00_name}_motor">
+        <hardwareInterface>hardware_interface/PositionJointInterface</hardwareInterface>
+        <mechanicalReduction>1</mechanicalReduction>
+    </actuator>
+</transmission>
+<transmission name="${link_01_name}_trans">
+    <type>transmission_interface/SimpleTransmission</type>
+    <joint name="${link_01_name}__${link_02_name}">
+        <hardwareInterface>hardware_interface/PositionJointInterface</hardwareInterface>
+    </joint>
+    <actuator name="${link_01_name}_motor">
+        <hardwareInterface>hardware_interface/PositionJointInterface</hardwareInterface>
+        <mechanicalReduction>1</mechanicalReduction>
+    </actuator>
+</transmission>
+<transmission name="${link_02_name}_trans">
+    <type>transmission_interface/SimpleTransmission</type>
+    <joint name="${link_02_name}__${link_02_name}">
+        <hardwareInterface>hardware_interface/PositionJointInterface</hardwareInterface>
+    </joint>
+    <actuator name="${link_02_name}_motor">
+        <hardwareInterface>hardware_interface/PositionJointInterface</hardwareInterface>
+        <mechanicalReduction>1</mechanicalReduction>
+    </actuator>
+</transmission>
+<transmission name="${link_03_name}_trans">
+    <type>transmission_interface/SimpleTransmission</type>
+    <joint name="${link_03_name}__${link_04_name}">
+        <hardwareInterface>hardware_interface/PositionJointInterface</hardwareInterface>
+    </joint>
+    <actuator name="${link_03_name}_motor">
+        <hardwareInterface>hardware_interface/PositionJointInterface</hardwareInterface>
+        <mechanicalReduction>1</mechanicalReduction>
+    </actuator>
+</transmission>
+<transmission name="${link_04_name}_trans">
+    <type>transmission_interface/SimpleTransmission</type>
+    <joint name="${link_04_name}__${link_05_name}">
+        <hardwareInterface>hardware_interface/PositionJointInterface</hardwareInterface>
+    </joint>
+    <actuator name="${link_04_name}_motor">
+        <hardwareInterface>hardware_interface/PositionJointInterface</hardwareInterface>
+        <mechanicalReduction>1</mechanicalReduction>
+    </actuator>
+</transmission>
+<!-- END joint controller gazebo -->
   <gazebo>
     <plugin name="gazebo_ros_control" filename="libgazebo_ros_control.so">
     </plugin>
   </gazebo>
+  <gazebo>
+    <plugin name="joint_state_publisher" filename="libgazebo_ros_joint_state_publisher.so">
+      <jointName>${link_00_name}__${link_01_name},${link_01_name}__${link_02_name} ,${link_02_name}__${link_03_name} ,${link_03_name}__${link_04_name} ,${link_04_name}__${link_05_name} </jointName>
+    </plugin>
+  </gazebo>
 </robot>
